Commit message: Update joint limits

File: src/yahboom_rosmaster/yahboom_rosmaster_description/urdf/mech/rosmaster_x3_plus_arm.urdf.xacro (robot description, xacro)
@@ -35,5 +35,5 @@
         <child link="${prefix}arm_link1"/>
         <axis xyz="0 0 -1"/>
-        <limit lower="-1.5708" upper="1.5708" effort="100" velocity="1"/>
+        <limit lower="-2" upper="2" effort="100" velocity="5"/>
     </joint>
     <link name="${prefix}arm_link2">
@@ -70,5 +70,5 @@
         <child link="${prefix}arm_link2"/>
         <axis xyz="0 0 -1"/>
-        <limit lower="-1.5708" upper="1.5708" effort="100" velocity="1"/>
+        <limit lower="-2" upper="2" effort="100" velocity="5"/>
     </joint>
     <link name="${prefix}arm_link3">
@@ -105,5 +105,5 @@
         <child link="${prefix}arm_link3"/>
         <axis xyz="0 0 -1"/>
-        <limit lower="-1.5708" upper="1.5708" effort="100" velocity="1"/>
+        <limit lower="-2.5" upper="2.5" effort="100" velocity="5"/>
     </joint>
     <link name="${prefix}arm_link4">
@@ -140,5 +140,5 @@
         <child link="${prefix}arm_link4"/>
         <axis xyz="0 0 -1"/>
-        <limit lower="-1.5708" upper="1.5708" effort="100" velocity="1"/>
+        <limit lower="-2.5" upper="2.5" effort="100" velocity="5"/>
     </joint>
     <link name="${prefix}arm_link5">
@@ -175,5 +175,5 @@
         <child link="${prefix}arm_link5"/>
         <axis xyz="0 0 1"/>
-        <limit lower="-1.5708" upper="3.14159" effort="100" velocity="1"/>
+        <limit lower="-2" upper="3.14159" effort="100" velocity="5"/>
     </joint>
     <link name="${prefix}rlink1">
