Commit message: arm: calibrate servo_map to the real 0-180deg = +/-pi/2 servo travel; tighten URDF limits
servo_map.yaml was still the Phase-0 placeholder, mapping the URDF's
fictional +/-2 rad (joints 1-2) and +/-2.5 rad (joints 3-4) ranges onto
the servos' 0-180 deg. That scales every commanded angle to ~79% / ~63%
of the requested motion, and the /joint_states readback inverts through
the same wrong map — so logs showed cmd==act while the physical arm
under-articulated. FK of the placeholder-distorted angles predicts the
fingertip lands ~16 cm above the model's belief at the logged pick pose,
matching the tape-measured miss (high and short) on hardware.

The real bus servos travel 0-180 deg with 90 deg = joint zero, i.e.
-pi/2..+pi/2 rad per joint. Map all five arm joints accordingly, and
tighten the URDF limits to +/-1.5708 so IK can no longer return angles
the bridge would silently clamp at the servo ends (this pick commanded
joint2=-1.73 rad, beyond physical travel).

Note: arm_joint5's zero moves from servo 70 deg to 90 deg (the old map
was asymmetric), so wrist-roll behavior shifts by 20 deg and the
previously-tuned grasp_roll_offset_rad=3.1416 now corresponds to
~1.5708 with the corrected map.

Co-Authored-By: Claude Fable 5 <noreply@anthropic.com>

File: src/yahboom_rosmaster/yahboom_rosmaster_description/urdf/mech/rosmaster_x3_plus_arm.urdf.xacro (robot description, xacro)
@@ -35,5 +35,5 @@
         <child link="${prefix}arm_link1"/>
         <axis xyz="0 0 -1"/>
-        <limit lower="-2" upper="2" effort="100" velocity="5"/>
+        <limit lower="-1.5708" upper="1.5708" effort="100" velocity="5"/>
     </joint>
     <link name="${prefix}arm_link2">
@@ -70,5 +70,5 @@
         <child link="${prefix}arm_link2"/>
         <axis xyz="0 0 -1"/>
-        <limit lower="-2" upper="2" effort="100" velocity="5"/>
+        <limit lower="-1.5708" upper="1.5708" effort="100" velocity="5"/>
     </joint>
     <link name="${prefix}arm_link3">
@@ -105,5 +105,5 @@
         <child link="${prefix}arm_link3"/>
         <axis xyz="0 0 -1"/>
-        <limit lower="-2.5" upper="2.5" effort="100" velocity="5"/>
+        <limit lower="-1.5708" upper="1.5708" effort="100" velocity="5"/>
     </joint>
     <link name="${prefix}arm_link4">
@@ -140,5 +140,5 @@
         <child link="${prefix}arm_link4"/>
         <axis xyz="0 0 -1"/>
-        <limit lower="-2.5" upper="2.5" effort="100" velocity="5"/>
+        <limit lower="-1.5708" upper="1.5708" effort="100" velocity="5"/>
     </joint>
     <link name="${prefix}arm_link5">
@@ -175,5 +175,5 @@
         <child link="${prefix}arm_link5"/>
         <axis xyz="0 0 1"/>
-        <limit lower="-2" upper="3.14159" effort="100" velocity="5"/>
+        <limit lower="-1.5708" upper="1.5708" effort="100" velocity="5"/>
     </joint>
     <link name="${prefix}rlink1">
