Commit message: MoveIt working with gazebo

File: src/yahboom_rosmaster/yahboom_rosmaster_description/urdf/control/rosmaster_x3_plus_ros2_control.urdf.xacro (robot description, xacro)
@@ -41,4 +41,39 @@
                 <state_interface name="velocity"/>
             </joint>
+            <joint name="${prefix}rlink_joint2">
+                <param name="mimic">${prefix}grip_joint</param>
+                <param name="multiplier">-1</param>
+                <command_interface name="position"/>
+                <state_interface name="position"/>
+                <state_interface name="velocity"/>
+            </joint>
+            <joint name="${prefix}rlink_joint3">
+                <param name="mimic">${prefix}grip_joint</param>
+                <param name="multiplier">1</param>
+                <command_interface name="position"/>
+                <state_interface name="position"/>
+                <state_interface name="velocity"/>
+            </joint>
+            <joint name="${prefix}llink_joint1">
+                <param name="mimic">${prefix}grip_joint</param>
+                <param name="multiplier">-1</param>
+                <command_interface name="position"/>
+                <state_interface name="position"/>
+                <state_interface name="velocity"/>
+            </joint>
+            <joint name="${prefix}llink_joint2">
+                <param name="mimic">${prefix}grip_joint</param>
+                <param name="multiplier">1</param>
+                <command_interface name="position"/>
+                <state_interface name="position"/>
+                <state_interface name="velocity"/>
+            </joint>
+            <joint name="${prefix}llink_joint3">
+                <param name="mimic">${prefix}grip_joint</param>
+                <param name="multiplier">-1</param>
+                <command_interface name="position"/>
+                <state_interface name="position"/>
+                <state_interface name="velocity"/>
+            </joint>
         </ros2_control>
     </xacro:macro>

Commit message: No llega al punto pero bien antes de eso

File: src/yahboom_rosmaster/yahboom_rosmaster_description/urdf/control/rosmaster_x3_plus_ros2_control.urdf.xacro (robot description, xacro)
@@ -1,5 +1,5 @@
 <?xml version="1.0" ?>
 <robot xmlns:xacro="http://wiki.ros.org/xacro">
-    <xacro:macro name="yahboom_rosmaster_x3_plus_ros2_control" params="prefix use_gazebo">
+    <xacro:macro name="yahboom_rosmaster_x3_plus_ros2_control" params="prefix use_gazebo include_mimic_control:=true">
         <ros2_control name="RobotSystem" type="system">
             <hardware>
@@ -41,39 +41,41 @@
                 <state_interface name="velocity"/>
             </joint>
-            <joint name="${prefix}rlink_joint2">
-                <param name="mimic">${prefix}grip_joint</param>
-                <param name="multiplier">-1</param>
-                <command_interface name="position"/>
-                <state_interface name="position"/>
-                <state_interface name="velocity"/>
-            </joint>
-            <joint name="${prefix}rlink_joint3">
-                <param name="mimic">${prefix}grip_joint</param>
-                <param name="multiplier">1</param>
-                <command_interface name="position"/>
-                <state_interface name="position"/>
-                <state_interface name="velocity"/>
-            </joint>
-            <joint name="${prefix}llink_joint1">
-                <param name="mimic">${prefix}grip_joint</param>
-                <param name="multiplier">-1</param>
-                <command_interface name="position"/>
-                <state_interface name="position"/>
-                <state_interface name="velocity"/>
-            </joint>
-            <joint name="${prefix}llink_joint2">
-                <param name="mimic">${prefix}grip_joint</param>
-                <param name="multiplier">1</param>
-                <command_interface name="position"/>
-                <state_interface name="position"/>
-                <state_interface name="velocity"/>
-            </joint>
-            <joint name="${prefix}llink_joint3">
-                <param name="mimic">${prefix}grip_joint</param>
-                <param name="multiplier">-1</param>
-                <command_interface name="position"/>
-                <state_interface name="position"/>
-                <state_interface name="velocity"/>
-            </joint>
+            <xacro:if value="${include_mimic_control}">
+                <joint name="${prefix}rlink_joint2">
+                    <param name="mimic">${prefix}grip_joint</param>
+                    <param name="multiplier">-1</param>
+                    <command_interface name="position"/>
+                    <state_interface name="position"/>
+                    <state_interface name="velocity"/>
+                </joint>
+                <joint name="${prefix}rlink_joint3">
+                    <param name="mimic">${prefix}grip_joint</param>
+                    <param name="multiplier">1</param>
+                    <command_interface name="position"/>
+                    <state_interface name="position"/>
+                    <state_interface name="velocity"/>
+                </joint>
+                <joint name="${prefix}llink_joint1">
+                    <param name="mimic">${prefix}grip_joint</param>
+                    <param name="multiplier">-1</param>
+                    <command_interface name="position"/>
+                    <state_interface name="position"/>
+                    <state_interface name="velocity"/>
+                </joint>
+                <joint name="${prefix}llink_joint2">
+                    <param name="mimic">${prefix}grip_joint</param>
+                    <param name="multiplier">1</param>
+                    <command_interface name="position"/>
+                    <state_interface name="position"/>
+                    <state_interface name="velocity"/>
+                </joint>
+                <joint name="${prefix}llink_joint3">
+                    <param name="mimic">${prefix}grip_joint</param>
+                    <param name="multiplier">-1</param>
+                    <command_interface name="position"/>
+                    <state_interface name="position"/>
+                    <state_interface name="velocity"/>
+                </joint>
+            </xacro:if>
         </ros2_control>
     </xacro:macro>

File: src/yahboom_rosmaster/yahboom_rosmaster_description/urdf/mech/rosmaster_x3_plus_arm.urdf.xacro (robot description, xacro)
@@ -35,5 +35,5 @@
         <child link="${prefix}arm_link1"/>
         <axis xyz="0 0 -1"/>
-        <limit lower="-1.5708" upper="1.5708" effort="100" velocity="1"/>
+        <limit lower="-2" upper="2" effort="100" velocity="5"/>
     </joint>
     <link name="${prefix}arm_link2">
@@ -70,5 +70,5 @@
         <child link="${prefix}arm_link2"/>
         <axis xyz="0 0 -1"/>
-        <limit lower="-1.5708" upper="1.5708" effort="100" velocity="1"/>
+        <limit lower="-2" upper="2" effort="100" velocity="5"/>
     </joint>
     <link name="${prefix}arm_link3">
@@ -105,5 +105,5 @@
         <child link="${prefix}arm_link3"/>
         <axis xyz="0 0 -1"/>
-        <limit lower="-1.5708" upper="1.5708" effort="100" velocity="1"/>
+        <limit lower="-2.5" upper="2.5" effort="100" velocity="5"/>
     </joint>
     <link name="${prefix}arm_link4">
@@ -140,5 +140,5 @@
         <child link="${prefix}arm_link4"/>
         <axis xyz="0 0 -1"/>
-        <limit lower="-1.5708" upper="1.5708" effort="100" velocity="1"/>
+        <limit lower="-2.5" upper="2.5" effort="100" velocity="5"/>
     </joint>
     <link name="${prefix}arm_link5">
@@ -175,5 +175,5 @@
         <child link="${prefix}arm_link5"/>
         <axis xyz="0 0 1"/>
-        <limit lower="-1.5708" upper="3.14159" effort="100" velocity="1"/>
+        <limit lower="-2" upper="3.14159" effort="100" velocity="5"/>
     </joint>
     <link name="${prefix}rlink1">

File: src/yahboom_rosmaster/yahboom_rosmaster_description/urdf/robots/rosmaster_x3_plus.urdf.xacro (robot description, xacro)
@@ -5,4 +5,5 @@
     <xacro:arg name="prefix" default=""/>
     <xacro:arg name="use_gazebo" default="false"/>
+    <xacro:arg name="include_mimic_control" default="true"/>
     <link name="$(arg prefix)base_footprint"/>
     <link name="$(arg prefix)base_link">
@@ -208,4 +209,5 @@
     <xacro:yahboom_rosmaster_x3_plus_ros2_control
       prefix="$(arg prefix)"
-      use_gazebo="$(arg use_gazebo)"/>
+      use_gazebo="$(arg use_gazebo)"
+      include_mimic_control="$(arg include_mimic_control)"/>
 </robot>

Commit message: wheeels

File: src/yahboom_rosmaster/yahboom_rosmaster_description/urdf/control/rosmaster_x3_plus_ros2_control.urdf.xacro (robot description, xacro)
@@ -11,4 +11,36 @@
                 </xacro:unless>
             </hardware>
+            <joint name="${prefix}front_left_wheel_joint">
+                <command_interface name="velocity">
+                    <param name="min">-50.0</param>
+                    <param name="max">50.0</param>
+                </command_interface>
+                <state_interface name="position"/>
+                <state_interface name="velocity"/>
+            </joint>
+            <joint name="${prefix}front_right_wheel_joint">
+                <command_interface name="velocity">
+                    <param name="min">-50.0</param>
+                    <param name="max">50.0</param>
+                </command_interface>
+                <state_interface name="position"/>
+                <state_interface name="velocity"/>
+            </joint>
+            <joint name="${prefix}back_left_wheel_joint">
+                <command_interface name="velocity">
+                    <param name="min">-50.0</param>
+                    <param name="max">50.0</param>
+                </command_interface>
+                <state_interface name="position"/>
+                <state_interface name="velocity"/>
+            </joint>
+            <joint name="${prefix}back_right_wheel_joint">
+                <command_interface name="velocity">
+                    <param name="min">-50.0</param>
+                    <param name="max">50.0</param>
+                </command_interface>
+                <state_interface name="position"/>
+                <state_interface name="velocity"/>
+            </joint>
             <joint name="${prefix}arm_joint1">
                 <command_interface name="position"/>

File: src/yahboom_rosmaster/yahboom_rosmaster_description/urdf/mech/mecanum_wheel.urdf.xacro (robot description, xacro)
@@ -7,5 +7,5 @@
   <xacro:property name="wheel_xoff" value="0.08" />
   <xacro:property name="wheel_yoff" value="-0.01" />
-  <xacro:macro name="mecanum_wheel" params="prefix side x_reflect y_reflect">
+  <xacro:macro name="mecanum_wheel" params="prefix side x_reflect y_reflect z_offset:=${-wheel_radius}">
     <link name="${prefix}${side}_wheel_link">
       <visual>
@@ -37,5 +37,5 @@
       <parent link="${prefix}base_link"/>
       <child link="${prefix}${side}_wheel_link"/>
-      <origin xyz="${x_reflect*wheel_xoff} ${y_reflect*(wheel_separation/2+wheel_yoff)} ${-wheel_radius}" rpy="0 0 0"/>
+      <origin xyz="${x_reflect*wheel_xoff} ${y_reflect*(wheel_separation/2+wheel_yoff)} ${z_offset}" rpy="0 0 0"/>
     </joint>
     <gazebo reference="${prefix}${side}_wheel_link">

File: src/yahboom_rosmaster/yahboom_rosmaster_description/urdf/robots/rosmaster_x3_plus.urdf.xacro (robot description, xacro)
@@ -199,8 +199,9 @@
         </gazebo>
     </xacro:if>
-    <xacro:include filename="$(find yahboom_rosmaster_description)/urdf/control/velocity_control_plugin.urdf.xacro" />
-    <xacro:load_velocity_control_plugin use_gazebo="$(arg use_gazebo)"/>
-    <xacro:include filename="$(find yahboom_rosmaster_description)/urdf/control/gz_odom_publisher.urdf.xacro" />
-    <xacro:load_gz_odom_publisher robot_name="$(arg robot_name)" use_gazebo="$(arg use_gazebo)"/>
+    <xacro:include filename="$(find yahboom_rosmaster_description)/urdf/mech/mecanum_wheel.urdf.xacro"/>
+    <xacro:mecanum_wheel prefix="$(arg prefix)" side="front_left"  x_reflect="1"  y_reflect="1"  z_offset="-0.076"/>
+    <xacro:mecanum_wheel prefix="$(arg prefix)" side="front_right" x_reflect="1"  y_reflect="-1" z_offset="-0.076"/>
+    <xacro:mecanum_wheel prefix="$(arg prefix)" side="back_left"   x_reflect="-1" y_reflect="1"  z_offset="-0.076"/>
+    <xacro:mecanum_wheel prefix="$(arg prefix)" side="back_right"  x_reflect="-1" y_reflect="-1" z_offset="-0.076"/>
     <xacro:include filename="$(find yahboom_rosmaster_description)/urdf/control/gazebo_sim_ros2_control.urdf.xacro" />
     <xacro:load_gazebo_sim_ros2_control_plugin
