Commit message: restore from before claude

File: src/yahboom_rosmaster/yahboom_rosmaster_description/urdf/control/gz_odom_publisher.urdf.xacro (robot description, xacro)
@@ -1,12 +1,18 @@
 <?xml version="1.0" ?>
 <robot xmlns:xacro="http://wiki.ros.org/xacro">
+    <!--
+      Publishes the model's ground-truth pose as nav_msgs/Odometry from Gazebo,
+      bridged to mecanum_drive_controller/odom by ros_gz_bridge so consumers
+      (executor closed-loop drive, EKF) work in both sim and real. Plugin
+      filename uses the Ignition Fortress (gz Sim 6) naming.
+    -->
     <xacro:macro name="load_gz_odom_publisher" params="robot_name use_gazebo">
         <xacro:if value="${use_gazebo}">
             <gazebo>
-                <plugin filename="gz-sim-odometry-publisher-system"
-                        name="gz::sim::systems::OdometryPublisher">
+                <plugin filename="ignition-gazebo-odometry-publisher-system"
+                        name="ignition::gazebo::systems::OdometryPublisher">
                     <odom_frame>odom</odom_frame>
                     <robot_base_frame>base_footprint</robot_base_frame>
-                    <odom_topic>/mecanum_drive_controller/odom</odom_topic>
+                    <odom_topic>/model/${robot_name}/odometry</odom_topic>
                     <dimensions>2</dimensions>
                     <odom_publish_frequency>50</odom_publish_frequency>

File: src/yahboom_rosmaster/yahboom_rosmaster_description/urdf/control/rosmaster_x3_plus_ros2_control.urdf.xacro (robot description, xacro)
@@ -11,36 +11,4 @@
                 </xacro:unless>
             </hardware>
-            <joint name="${prefix}front_left_wheel_joint">
-                <command_interface name="velocity">
-                    <param name="min">-50.0</param>
-                    <param name="max">50.0</param>
-                </command_interface>
-                <state_interface name="position"/>
-                <state_interface name="velocity"/>
-            </joint>
-            <joint name="${prefix}front_right_wheel_joint">
-                <command_interface name="velocity">
-                    <param name="min">-50.0</param>
-                    <param name="max">50.0</param>
-                </command_interface>
-                <state_interface name="position"/>
-                <state_interface name="velocity"/>
-            </joint>
-            <joint name="${prefix}back_left_wheel_joint">
-                <command_interface name="velocity">
-                    <param name="min">-50.0</param>
-                    <param name="max">50.0</param>
-                </command_interface>
-                <state_interface name="position"/>
-                <state_interface name="velocity"/>
-            </joint>
-            <joint name="${prefix}back_right_wheel_joint">
-                <command_interface name="velocity">
-                    <param name="min">-50.0</param>
-                    <param name="max">50.0</param>
-                </command_interface>
-                <state_interface name="position"/>
-                <state_interface name="velocity"/>
-            </joint>
             <joint name="${prefix}arm_joint1">
                 <command_interface name="position"/>

File: src/yahboom_rosmaster/yahboom_rosmaster_description/urdf/robots/rosmaster_x3_plus.urdf.xacro (robot description, xacro)
@@ -21,5 +21,5 @@
             <origin xyz="0 0 0" rpy="0 0 0"/>
             <geometry>
-                <mesh filename="file://$(find yahboom_rosmaster_description)/meshes/rosmaster_x3/visual/base_link_X3.STL"/>
+                <mesh filename="file://$(find yahboom_rosmaster_description)/meshes/rosmaster_x3_plus/visual/base_link.STL"/>
             </geometry>
             <material name="x3_plus_green">
@@ -28,7 +28,7 @@
         </visual>
         <collision>
-            <origin xyz="0 0 0.06" rpy="0 0 0"/>
-            <geometry>
-                <box size="0.20 0.16 0.10"/>
+            <origin xyz="0 0 0" rpy="0 0 0"/>
+            <geometry>
+                <mesh filename="file://$(find yahboom_rosmaster_description)/meshes/rosmaster_x3_plus/collision/base_link.STL"/>
             </geometry>
         </collision>
@@ -199,9 +199,8 @@
         </gazebo>
     </xacro:if>
-    <xacro:include filename="$(find yahboom_rosmaster_description)/urdf/mech/mecanum_wheel.urdf.xacro"/>
-    <xacro:mecanum_wheel prefix="$(arg prefix)" side="front_left"  x_reflect="1"  y_reflect="1"  z_offset="-0.0435"/>
-    <xacro:mecanum_wheel prefix="$(arg prefix)" side="front_right" x_reflect="1"  y_reflect="-1" z_offset="-0.0435"/>
-    <xacro:mecanum_wheel prefix="$(arg prefix)" side="back_left"   x_reflect="-1" y_reflect="1"  z_offset="-0.0435"/>
-    <xacro:mecanum_wheel prefix="$(arg prefix)" side="back_right"  x_reflect="-1" y_reflect="-1" z_offset="-0.0435"/>
+    <xacro:include filename="$(find yahboom_rosmaster_description)/urdf/control/velocity_control_plugin.urdf.xacro" />
+    <xacro:load_velocity_control_plugin use_gazebo="$(arg use_gazebo)"/>
+    <xacro:include filename="$(find yahboom_rosmaster_description)/urdf/control/gz_odom_publisher.urdf.xacro" />
+    <xacro:load_gz_odom_publisher robot_name="$(arg robot_name)" use_gazebo="$(arg use_gazebo)"/>
     <xacro:include filename="$(find yahboom_rosmaster_description)/urdf/control/gazebo_sim_ros2_control.urdf.xacro" />
     <xacro:load_gazebo_sim_ros2_control_plugin
