Commit message: better perception

File: src/yahboom_rosmaster/yahboom_rosmaster_description/urdf/robots/rosmaster_x3_plus.urdf.xacro (robot description, xacro)
@@ -89,5 +89,5 @@
     </link>
     <joint name="$(arg prefix)astra_joint" type="fixed">
-        <origin xyz="-0.043645 0 0.41955" rpy="0 0 0"/>
+        <origin xyz="-0.043645 0 0.41955" rpy="0 0.65 0"/>
         <parent link="$(arg prefix)base_link"/>
         <child link="$(arg prefix)camera_link"/>

Commit message: wheeels4

File: src/yahboom_rosmaster/yahboom_rosmaster_description/urdf/robots/rosmaster_x3_plus.urdf.xacro (robot description, xacro)
@@ -21,5 +21,5 @@
             <origin xyz="0 0 0" rpy="0 0 0"/>
             <geometry>
-                <mesh filename="file://$(find yahboom_rosmaster_description)/meshes/rosmaster_x3_plus/visual/base_link.STL"/>
+                <mesh filename="file://$(find yahboom_rosmaster_description)/meshes/rosmaster_x3/visual/base_link_X3.STL"/>
             </geometry>
             <material name="x3_plus_green">
@@ -28,7 +28,7 @@
         </visual>
         <collision>
-            <origin xyz="0 0 0" rpy="0 0 0"/>
-            <geometry>
-                <mesh filename="file://$(find yahboom_rosmaster_description)/meshes/rosmaster_x3_plus/collision/base_link.STL"/>
+            <origin xyz="0 0 0.06" rpy="0 0 0"/>
+            <geometry>
+                <box size="0.20 0.16 0.10"/>
             </geometry>
         </collision>

Commit message: Posicion robot y camara

File: src/yahboom_rosmaster/yahboom_rosmaster_description/urdf/robots/rosmaster_x3_plus.urdf.xacro (robot description, xacro)
@@ -89,5 +89,5 @@
     </link>
     <joint name="$(arg prefix)astra_joint" type="fixed">
-        <origin xyz="-0.043645 0 0.41955" rpy="0 0.65 0"/>
+        <origin xyz="-0.043645 0 0.41955" rpy="0 0.3316 0"/>
         <parent link="$(arg prefix)base_link"/>
         <child link="$(arg prefix)camera_link"/>
